Commit message: tirei o innorder

File: mobot_urdf/urdf/add_lidar.xacro (robot description, xacro)
@@ -25,12 +25,12 @@
           <inertia ixx="0.01" ixy="0" ixz="0" iyy="0.01" iyz="0" izz="0.01" />
       </inertial>
+      <joint name="lidar_joint" type="fixed">
+        <axis xyz="0 1 0" />
+        <origin xyz="0.1 0 0.56" rpy="0 0 0"/>
+        <parent link="base_link"/>
+        <child link="lidar_link"/>
+      </joint>
   </link>
   <!--the above displays a box meant to imply Lidar-->
-  <joint name="lidar_joint" type="fixed">
-      <axis xyz="0 1 0" />
-      <origin xyz="0.1 0 0.56" rpy="0 0 0"/>
-      <parent link="base_link"/>
-      <child link="lidar_link"/>
-  </joint>
     <!-- here is the gazebo plug-in to simulate a lidar sensor -->
   <gazebo reference="lidar_link">
